Commit message: Added control

File: autonomous_robot_description/urdf/autonomous_robot.urdf.xacro (robot description, xacro)
@@ -5,4 +5,6 @@
     <xacro:include filename="lidar.xacro" />
     <xacro:include filename="camera.xacro" />
-    <xacro:include filename="autonomous_robot_gazebo.xacro" />
+    <!-- <xacro:include filename="autonomous_robot_gazebo.xacro" /> -->
+    <xacro:include filename="ros2_control.xacro" />
+    <xacro:include filename="gazebo_color.xacro" />
 </robot>

File: autonomous_robot_description/urdf/autonomous_robot_gazebo.xacro (robot description, xacro)
@@ -1,31 +1,4 @@
 <?xml version="1.0"?>
 <robot xmlns:xacro="http://www.ros.org/wiki/xacro">
-    <gazebo reference="base_footprint">
-        <material>Gazebo/Black</material>
-    </gazebo>
-    <gazebo reference="base_link">
-        <material>Gazebo/Green</material>
-    </gazebo>
-    <gazebo reference="left_wheel_link">
-        <material>Gazebo/Blue</material>
-    </gazebo>
-    <gazebo reference="right_wheel_link">
-        <material>Gazebo/Blue</material>
-    </gazebo>
-    <gazebo reference="front_hinge">
-        <material>Gazebo/Grey</material>
-    </gazebo>
-    <gazebo reference="front_wheel_link">
-        <material>Gazebo/Blue</material>
-    </gazebo>
-    <gazebo reference="rear_hinge">
-        <material>Gazebo/Grey</material>
-    </gazebo>
-    <gazebo reference="rear_wheel_link">
-        <material>Gazebo/Blue</material>
-    </gazebo>
-    <gazebo reference="lidar_link">
-        <material>Gazebo/Purple</material>
-    </gazebo>
     <gazebo>
         <plugin name="gazebo_ros_diff_drive" filename="libgazebo_ros_diff_drive.so">

File: autonomous_robot_description/urdf/lidar.xacro (robot description, xacro)
@@ -27,9 +27,9 @@
             <pose> 0 0 0 0 0 0 </pose>
             <visualize>true</visualize>
-            <update_rate>10.0</update_rate>
+            <update_rate>5.0</update_rate>
             <ray>
                 <scan>
                     <horizontal>
-                        <samples>360</samples>
+                        <samples>90</samples>
                         <min_angle>-3.14</min_angle>
                         <max_angle>3.14</max_angle>
