Commit message: Saving changes before checkout

File: autonomous_robot_description/urdf/lidar.xacro (robot description, xacro)
@@ -13,5 +13,5 @@
         <collision>
             <geometry>
-                <box radius="${lidar_radius}" length="${lidar_h}" />
+                <cylinder radius="${lidar_radius}" length="${lidar_h}" />
             </geometry>
         </collision>
@@ -27,5 +27,5 @@
             <pose> 0 0 0 0 0 0 </pose>
             <visualize>true</visualize>
-            <update_rate>5.0</update_rate>
+            <update_rate>10.0</update_rate>
             <ray>
                 <scan>

File: autonomous_robot_description/urdf/ros2_control.xacro (robot description, xacro)
@@ -1,60 +1,28 @@
 <?xml version="1.0"?>
 <robot xmlns:xacro="http://www.ros.org/wiki/xacro">
-    <xacro:unless value="$(arg sim_mode)">
-        <ros2_control name="RealRobot" type="system">
-            <hardware>
-                <plugin>diffdrive_arduino/DiffDriveArduino</plugin>
-                <param name="left_wheel_name">left_wheel_joint</param>
-                <param name="right_wheel_name">right_wheel_joint</param>
-                <param name="loop_rate">30</param>
-                <param name="device">/dev/ttyUSB0</param>
-                <param name="baud_rate">57600</param>
-                <param name="timeout">1000</param>
-                <param name="enc_counts_per_rev">3436</param>
-            </hardware>
-            <joint name="left_wheel_joint">
-                <command_interface name="velocity">
-                    <param name="min">-10</param>
-                    <param name="max">10</param>
-                </command_interface>
-                <state_interface name="velocity"/>
-                <state_interface name="position"/>
-            </joint>
-            <joint name="right_wheel_joint">
-                <command_interface name="velocity">
-                    <param name="min">-10</param>
-                    <param name="max">10</param>
-                </command_interface>
-                <state_interface name="velocity"/>
-                <state_interface name="position"/>
-            </joint>
-        </ros2_control>
-    </xacro:unless>
-    <xacro:if value="$(arg sim_mode)">
-        <ros2_control name="GazeboSystem" type="system">
-            <hardware>
-                <plugin>gazebo_ros2_control/GazeboSystem</plugin>
-            </hardware>
-            <joint name="left_wheel_joint">
-                <command_interface name="velocity">
-                    <param name="min">-10</param>
-                    <param name="max">10</param>
-                </command_interface>
-                <state_interface name="velocity"/>
-                <state_interface name="position"/>
-            </joint>
-            <joint name="right_wheel_joint">
-                <command_interface name="velocity">
-                    <param name="min">-10</param>
-                    <param name="max">10</param>
-                </command_interface>
-                <state_interface name="velocity"/>
-                <state_interface name="position"/>
-            </joint>
-        </ros2_control>
-    </xacro:if>
+    <ros2_control name="GazeboSystem" type="system">
+        <hardware>
+            <plugin>gazebo_ros2_control/GazeboSystem</plugin>
+        </hardware>
+        <joint name="left_wheel_joint">
+            <command_interface name="velocity">
+                <param name="min">-10</param>
+                <param name="max">10</param>
+            </command_interface>
+            <state_interface name="velocity"/>
+            <state_interface name="position"/>
+        </joint>
+        <joint name="right_wheel_joint">
+            <command_interface name="velocity">
+                <param name="min">-10</param>
+                <param name="max">10</param>
+            </command_interface>
+            <state_interface name="velocity"/>
+            <state_interface name="position"/>
+        </joint>
+    </ros2_control>
     <gazebo>
         <plugin name="gazebo_ros2_control" filename="libgazebo_ros2_control.so">
-            <parameters>$(find autonomous_robot_description)/config/joint_controller.yaml</parameters>
+            <parameters>$(find autonomous_robot_description)/config/sim_joint_controller.yaml</parameters>
         </plugin>
     </gazebo>

File: install/autonomous_robot_description/share/autonomous_robot_description/urdf/autonomous_robot.urdf.xacro (robot description, xacro)
@@ -1,16 +1 @@
-<?xml version="1.0"?>
-<robot name="autonomous_robot" xmlns:xacro="http://www.ros.org/wiki/xacro">
-    <xacro:arg name="use_ros2_control" default="true"/>
-    <xacro:arg name="sim_mode" default="true"/>
-    <xacro:include filename="common_properties.xacro" />
-    <xacro:include filename="mobile_robot.xacro" />
-    <xacro:if value="$(arg use_ros2_control)"> <!--switching between ros2_control and gazebo control-->
-        <xacro:include filename="ros2_control.xacro" />
-    </xacro:if>
-    <xacro:unless value="$(arg use_ros2_control)">
-        <xacro:include filename="autonomous_robot_gazebo.xacro" />
-    </xacro:unless>
-    <xacro:include filename="lidar.xacro" />
-    <xacro:include filename="camera.xacro" />
-    <xacro:include filename="gazebo_color.xacro" />
-</robot>
+/home/tamir/autonomous_robot/autonomous_robot_description/urdf/autonomous_robot.urdf.xacro

File: install/autonomous_robot_description/share/autonomous_robot_description/urdf/autonomous_robot_gazebo.xacro (robot description, xacro)
@@ -1,27 +1 @@
-<?xml version="1.0"?>
-<robot xmlns:xacro="http://www.ros.org/wiki/xacro">
-    <gazebo>
-        <plugin name="gazebo_ros_diff_drive" filename="libgazebo_ros_diff_drive.so">
-            <!-- Update rate in Hz -->
-            <update_rate>50</update_rate>
-            <!-- wheels -->
-            <left_joint>left_wheel_joint</left_joint>
-            <right_joint>right_wheel_joint</right_joint>
-            <!-- kinematics -->
-            <wheel_separation>0.7</wheel_separation>
-            <wheel_diameter>0.16</wheel_diameter>
-            <!-- limits -->
-            <max_wheel_torque>200</max_wheel_torque>
-            <max_wheel_acceleration>10</max_wheel_acceleration>
-            <!-- input -->
-            <command_topic>cmd_vel</command_topic>
-            <!-- output -->
-            <publish_odom>true</publish_odom>
-            <publish_odom_tf>true</publish_odom_tf>
-            <publish_wheel_tf>true</publish_wheel_tf>
-            <odometry_topic>odom</odometry_topic>
-            <odometry_frame>odom</odometry_frame>
-            <robot_base_frame>base_footprint</robot_base_frame>
-        </plugin>
-    </gazebo>
-</robot>
+/home/tamir/autonomous_robot/autonomous_robot_description/urdf/autonomous_robot_gazebo.xacro

File: install/autonomous_robot_description/share/autonomous_robot_description/urdf/camera.xacro (robot description, xacro)
@@ -1,62 +1 @@
-<?xml version="1.0"?>
-<robot xmlns:xacro="http://www.ros.org/wiki/xacro">
-    <!-- Define Xacro properties -->
-    <xacro:property name="camera_l" value="0.01" />
-    <xacro:property name="camera_w" value="0.1" />
-    <xacro:property name="camera_h" value="0.05" />
-    <xacro:property name="base_l" value="1.0" />
-    <xacro:property name="base_h" value="0.3" />
-    <!-- Camera Link -->
-    <link name="camera_link">
-        <visual>
-            <geometry>
-                <box size="${camera_l} ${camera_w} ${camera_h}" />
-            </geometry>
-            <material name="red" />
-        </visual>
-        <collision>
-            <geometry>
-                <box size="${camera_l} ${camera_w} ${camera_h}" />
-            </geometry>
-        </collision>
-        <xacro:box_inertia mass="0.1" l="${camera_l}" w="${camera_w}" h="${camera_h}" xyz="0 0 0" rpy="0 0 0" />
-    </link>
-    <!-- Joint connecting base_link to camera_link -->
-    <joint name="base_camera_joint" type="fixed">
-        <parent link="base_link" />
-        <child link="camera_link" />
-        <origin xyz="${(base_l + camera_l) / 2.0} 0 ${(base_h / 2.0) - (camera_h / 2.0)}" rpy="0 0 0" />
-    </joint>
-    <!-- Camera Optical Link -->
-    <link name="camera_link_optical" />
-    <!-- Joint connecting camera_link to camera_link_optical -->
-    <joint name="camera_optical_joint" type="fixed">
-        <parent link="camera_link" />
-        <child link="camera_link_optical" />
-        <origin xyz="0 0 0" rpy="${-pi/2} 0 ${-pi/2}" />
-    </joint>
-    <!-- Gazebo Plugin (commented out correctly) -->
-    <gazebo reference="camera_link">
-        <material>Gazebo/Red</material>
-        <sensor name="camera_sensor" type="camera">
-            <pose>0 0 0 0 0 0</pose>
-            <visualize>true</visualize>
-            <update_rate>10.0</update_rate>
-            <camera>
-                <horizontal_fov>1.047</horizontal_fov>
-                <image>
-                    <format>B8G8R8</format>
-                    <width>640</width>
-                    <height>480</height>
-                </image>
-                <clip>
-                    <near>0.05</near>
-                    <far>8.0</far>
-                </clip>
-            </camera>
-            <plugin name="camera_controller" filename="libgazebo_ros_camera.so">
-                <frame_name>camera_link_optical</frame_name>
-            </plugin>
-        </sensor>
-    </gazebo>
-</robot>
+/home/tamir/autonomous_robot/autonomous_robot_description/urdf/camera.xacro

File: install/autonomous_robot_description/share/autonomous_robot_description/urdf/common_properties.xacro (robot description, xacro)
@@ -1,45 +1 @@
-<?xml version="1.0"?>
-<robot xmlns:xacro="http://www.ros.org/wiki/xacro">
-    <material name="grey">
-        <color rgba="0.5 0.5 0.5 1" />
-    </material>
-    <material name="green">
-        <color rgba="0 0.5 0 1" />
-    </material>
-    <material name="blue">
-        <color rgba="0 0 1 1" />
-    </material>
-    <material name="pink">
-        <color rgba="1 0 1 1" />
-    </material>
-    <material name="yellow">
-        <color rgba="0.5 0.5 0 1" />
-    </material>
-    <material name="orange">
-        <color rgba="1 0.5 0 1" />
-    </material>
-    <material name="red">
-        <color rgba="1 0 0.2 1" />
-    </material>
-    <material name="black">
-        <color rgba="0 0 0 1" />
-    </material>
-    <xacro:macro name="box_inertia" params="mass l w h xyz rpy">
-        <inertial>
-            <origin xyz="${xyz}" rpy="0 0 0" />
-            <mass value="${mass}" />
-            <inertia ixx="${mass/12 * (h*h + l*l)}" ixy="0" ixz="0"
-                     iyy="${mass/12 * (w*w + l*l)}" iyz="0"
-                     izz="${mass/12 * (h*h + w*w)}" />
-        </inertial>
-    </xacro:macro>
-    <xacro:macro name="wheel_inertia" params="mass l r xyz rpy">
-        <inertial>
-            <origin xyz="${xyz}" rpy="${rpy}" />
-            <mass value="${mass}" />
-            <inertia ixx="${mass/12 * (3*r*r + l*l)}" ixy="0" ixz="0"
-                     iyy="${mass/12 * (3*r*r + l*l)}" iyz="0"
-                     izz="${mass/2 * (r*r)}" />
-        </inertial>
-    </xacro:macro>
-</robot>
+/home/tamir/autonomous_robot/autonomous_robot_description/urdf/common_properties.xacro

File: install/autonomous_robot_description/share/autonomous_robot_description/urdf/gazebo_color.xacro (robot description, xacro)
@@ -1,30 +1 @@
-<?xml version="1.0"?>
-<robot xmlns:xacro="http://www.ros.org/wiki/xacro">
-    <gazebo reference="base_footprint">
-        <material>Gazebo/Black</material>
-    </gazebo>
-    <gazebo reference="base_link">
-        <material>Gazebo/Green</material>
-    </gazebo>
-    <gazebo reference="left_wheel_link">
-        <material>Gazebo/Blue</material>
-    </gazebo>
-    <gazebo reference="right_wheel_link">
-        <material>Gazebo/Blue</material>
-    </gazebo>
-    <gazebo reference="front_hinge">
-        <material>Gazebo/Grey</material>
-    </gazebo>
-    <gazebo reference="front_wheel_link">
-        <material>Gazebo/Blue</material>
-    </gazebo>
-    <gazebo reference="rear_hinge">
-        <material>Gazebo/Grey</material>
-    </gazebo>
-    <gazebo reference="rear_wheel_link">
-        <material>Gazebo/Blue</material>
-    </gazebo>
-    <gazebo reference="lidar_link">
-        <material>Gazebo/Purple</material>
-    </gazebo>
-</robot>
+/home/tamir/autonomous_robot/autonomous_robot_description/urdf/gazebo_color.xacro

File: install/autonomous_robot_description/share/autonomous_robot_description/urdf/lidar.xacro (robot description, xacro)
@@ -1,53 +1 @@
-<?xml version="1.0"?>
-<robot xmlns:xacro="http://www.ros.org/wiki/xacro">
-    <xacro:property name="lidar_radius" value="0.10" /><!--   was 0.05       -->
-    <xacro:property name="lidar_h" value="0.07" /> <!--   was 0.04       -->
-    <!--   Lidar        -->
-    <link name="lidar_link">
-        <visual>
-            <geometry>
-                <cylinder radius="${lidar_radius}" length="${lidar_h}" />
-            </geometry>
-            <material name="pink" />
-        </visual>
-        <collision>
-            <geometry>
-                <box radius="${lidar_radius}" length="${lidar_h}" />
-            </geometry>
-        </collision>
-        <xacro:wheel_inertia mass="0.1" l="${2*lidar_h}" r="${2*lidar_radius}" xyz="0 0 0" rpy="0 0 0" />
-    </link>
-    <joint name="base_lidar_joint" type="fixed">
-        <parent link="base_link" />
-        <child link="lidar_link" />
-        <origin xyz="${base_l / 4.0} 0 ${(base_h / 2.0) + (lidar_h / 2.0)}" rpy="0 0 0" />
-    </joint>
-    <gazebo reference ="lidar_link">
-        <sensor name="laser_link" type="ray">
-            <pose> 0 0 0 0 0 0 </pose>
-            <visualize>true</visualize>
-            <update_rate>5.0</update_rate>
-            <ray>
-                <scan>
-                    <horizontal>
-                        <samples>90</samples>
-                        <min_angle>-3.14</min_angle>
-                        <max_angle>3.14</max_angle>
-                    </horizontal>
-                </scan>
-                <range>
-                    <min>0.3</min>
-                    <max>10</max>
-                </range>
-            </ray>
-            <plugin name="laser_controller" filename="libgazebo_ros_ray_sensor.so">
-                <ros>
-                    <argument>~/out:=scan</argument> <!--   the topic we are publishing on    -->
-                </ros>
-                <output_type>sensor_msgs/LaserScan</output_type>
-                <frame_name>lidar_link</frame_name>
-            </plugin>
-        </sensor>
-    </gazebo>
-    <!-- ${-(pi) / 12.0 * 11} = -2.87979327-->
-</robot>
+/home/tamir/autonomous_robot/autonomous_robot_description/urdf/lidar.xacro

File: install/autonomous_robot_description/share/autonomous_robot_description/urdf/mobile_robot.xacro (robot description, xacro)
@@ -1,156 +1 @@
-<?xml version="1.0"?>
-<robot xmlns:xacro="http://www.ros.org/wiki/xacro">
-    <xacro:property name="wheel_r" value="0.16" /> <!-- without load the wheel diameter is 0.35 (radius = 0.175) so might go between 0.16 - 0.17 with standard load -->
-    <xacro:property name="wheel_l" value="0.16" />
-    <xacro:property name="wheel_axis_h" value="0.18802" />
-    <xacro:property name="hinge_l" value="${wheel_r - small_wheel_r + wheel_axis_h}" />
-    <xacro:property name="hinge_r" value="0.02" />
-    <xacro:property name="small_wheel_r" value="0.063" />
-    <xacro:property name="small_wheel_l" value="0.028" />
-    <xacro:property name="axis_dist" value="0.03" />
-    <xacro:property name="base_l" value="1.0" />
-    <xacro:property name="base_w" value="0.7" />
-    <xacro:property name="base_h" value="0.3" />
-    <xacro:property name="base_xyz" value="0 0 0" /> <!-- ${base_h / 2} : what z used to be -->
-    <xacro:property name="wheel_rpy" value="${pi / 2.0} 0 0" />
-    <xacro:property name="camera_l" value="0.01" />
-    <xacro:property name="camera_w" value="0.1" />
-    <xacro:property name="camera_h" value="0.05" />
-    <!-- body -->
-    <link name="base_footprint" />
-    <link name="base_link">
-        <visual>
-            <geometry>
-                <box size="${base_l} ${base_w} ${base_h}" />
-            </geometry>
-            <origin xyz="${base_xyz}" rpy="0 0 0" />
-            <material name="green" />
-        </visual>
-        <collision>
-            <geometry>
-                <box size="${base_l} ${base_w} ${base_h}" />
-            </geometry>
-            <origin xyz="${base_xyz}" rpy="0 0 0" />
-        </collision>
-        <xacro:box_inertia mass="25.0" l="${2*base_l}" w="${2*base_w}" h="${2*base_h}" xyz="${base_xyz}" rpy="0 0 0" />
-    </link>
-    <joint name="footprint_base_joint" type="fixed">
-        <parent link="base_footprint" />
-        <child link="base_link" />
-        <origin xyz="0 0 ${wheel_r + wheel_axis_h + (base_h / 2.0)}" rpy="0 0 0" /> <!-- + (base_h / 2) -->
-    </joint>
-    <!-- wheel funtions -->
-    <xacro:macro name="create_wheel_link" params="prefix">
-    <link name="${prefix}_wheel_link">
-        <visual>
-            <geometry>
-                <cylinder radius="${wheel_r}" length="${wheel_l}" />
-            </geometry>
-            <origin xyz="0 0 0" rpy="${wheel_rpy}" />
-            <material name="blue" />
-        </visual>
-        <collision>
-            <geometry>
-                <cylinder radius="${wheel_r}" length="${wheel_l}" />
-            </geometry>
-            <origin xyz="0 0 0" rpy="${wheel_rpy}" />
-        </collision>
-        <xacro:wheel_inertia mass="3.0" l="${2*wheel_l}" r="${2*wheel_r}" xyz="0 0 0" rpy="${wheel_rpy}" />
-    </link>
-    </xacro:macro>
-    <xacro:macro name="create_small_wheel_link" params="prefix">
-    <link name="${prefix}_wheel_link">
-        <visual>
-            <geometry>
-                <cylinder radius="${small_wheel_r}" length="${small_wheel_l}" />
-            </geometry>
-            <origin xyz="0 0 0" rpy="${wheel_rpy}" />
-            <material name="blue" />
-        </visual>
-        <collision>
-            <geometry>
-                <cylinder radius="${small_wheel_r}" length="${small_wheel_l}" />
-            </geometry>
-            <origin xyz="0 0 0" rpy="${wheel_rpy}" />
-        </collision>
-        <xacro:wheel_inertia mass="1.5" l="${2*small_wheel_l}" r="${2*small_wheel_r}" xyz="0 0 0" rpy="${wheel_rpy}" />
-    </link>
-    </xacro:macro>
-    <!-- wheels creations -->
-    <xacro:create_wheel_link prefix="left" />
-    <joint name="left_wheel_joint" type="continuous">
-        <parent link="base_link" />
-        <child link="left_wheel_link" />
-        <origin xyz="0 ${(base_w - wheel_r) / 2} ${-(base_h / 2) - wheel_axis_h}" rpy="0 0 0" />
-        <axis xyz="0 1 0" />
-        <limit velocity="100.0" effort="100.0" />
-        <!-- <dynamics damping="10.0" friction="10.0" /> that's actually a lot prettyh sureeee -->
-    </joint>
-    <xacro:create_wheel_link prefix="right" />
-    <joint name="right_wheel_joint" type="continuous">
-        <parent link="base_link" />
-        <child link="right_wheel_link" />
-        <origin xyz="0 ${-((base_w - wheel_r) / 2)} ${-(base_h / 2) - wheel_axis_h}" rpy="0 0 0" />
-         <axis xyz="0 1 0" />
-    </joint>
-    <!-- Front -->
-    <link name="front_hinge">
-        <visual>
-            <geometry>
-                <cylinder radius="${hinge_r}" length="${hinge_l}" />
-            </geometry>
-            <origin xyz="0 0 ${hinge_l / 2.0}" rpy="0 0 0" />
-            <material name="grey" />
-        </visual>
-        <collision>
-            <geometry>
-                <cylinder radius="${hinge_r}" length="${hinge_l}" />
-            </geometry>
-            <origin xyz="0 0 ${hinge_l / 2.0}" rpy="0 0 0" />
-        </collision>
-        <xacro:wheel_inertia mass="0.5" l="${2*hinge_l}" r="${2*hinge_r}" xyz="0 0 ${hinge_l / 2.0}" rpy="0 0 0" />
-    </link>
-    <joint name="front_hinge_joint" type="continuous">
-        <parent link="base_link" />
-        <child link="front_hinge" />
-        <origin xyz="0.48 0 ${-((base_h / 2.0) + wheel_r - small_wheel_r + wheel_axis_h)}" rpy="0 0 0" />
-        <axis xyz="0 0 1" />
-    </joint>
-    <xacro:create_small_wheel_link prefix="front" />
-    <joint name="front_wheel_joint" type="continuous">
-        <parent link="front_hinge" />
-        <child link="front_wheel_link" />
-        <origin xyz="${-axis_dist} 0 0" rpy="0 0 0" />
-        <axis xyz="0 1 0" />
-    </joint>
-    <!-- Rear -->
-    <link name="rear_hinge">
-        <visual>
-            <geometry>
-                <cylinder radius="${hinge_r}" length="${hinge_l}" />
-            </geometry>
-            <origin xyz="0 0 ${(hinge_l) / 2.0}" rpy="0 0 0" />
-            <material name="grey" />
-        </visual>
-        <collision>
-            <geometry>
-                <cylinder radius="${hinge_r}" length="${hinge_l}" />
-            </geometry>
-            <origin xyz="0 0 ${(hinge_l) / 2.0}" rpy="0 0 0" />
-        </collision>
-        <xacro:wheel_inertia mass="0.5" l="${2*hinge_l}" r="${2*hinge_r}" xyz="0 0 ${(hinge_l) / 2.0}" rpy="0 0 0" />
-    </link>
-    <joint name="rear_hinge_joint" type="continuous">
-        <parent link="base_link" />
-        <child link="rear_hinge" />
-        <origin xyz="-0.48 0 ${-((base_h / 2) + wheel_r - small_wheel_r + wheel_axis_h)}" rpy="0 0 0" />
-        <axis xyz="0 0 1" />
-    </joint>
-    <xacro:create_small_wheel_link prefix="rear" />
-    <joint name="rear_wheel_joint" type="continuous">
-        <parent link="rear_hinge" />
-        <child link="rear_wheel_link" />
-        <origin xyz="${-axis_dist} 0 0" rpy="0 0 0" />
-         <axis xyz="0 1 0" />
-    </joint>
-</robot>
+/home/tamir/autonomous_robot/autonomous_robot_description/urdf/mobile_robot.xacro
